Commit message: add 4 arms

File: urdf/arm.xacro (robot description, xacro)
@@ -27,112 +27,114 @@
   </xacro:macro>
   <!-- Begin arm joints and links -->
-  <link name="arm_base">
-    <visual>
-      <origin rpy="0.0 0 0" xyz="0 0 0.0"/>
-      <geometry>
-        <box size="${arm_base_width} ${arm_base_width} ${arm_base_height}"/>
-      </geometry>
-    </visual>
-    <xacro:box_inertial mass="${arm_mass}" length="${arm_base_width}" width="${arm_base_width}" heigth="${arm_base_height}"/>
-    <buoyancy><compensation>1.0</compensation></buoyancy>
-  </link>
-  <joint name="base_link_to_arm_base" type="fixed">
-    <parent link="base_link"/>
-    <child link="arm_base"/>
-    <origin rpy="0 0 0" xyz="0 0 0.9"/>
-  </joint>
-  <link name="arm_hand">
-    <visual>
-      <origin rpy="0 0 0" xyz="0 0 ${arm_hand_length/2}"/>
-      <geometry>
-        <cylinder radius="${arm_hand_width}" length="${arm_hand_length}"/>
-      </geometry>
-    </visual>
-    <collision>
-      <origin rpy="0 0 0" xyz="0 0 ${arm_hand_length/2}"/>
-      <geometry>
-        <cylinder radius="${arm_hand_width}" length="${arm_hand_length}"/>
-      </geometry>
-    </collision>
-    <inertial>
-      <origin rpy="0 0 0" xyz="0 0 ${arm_hand_length/2}"/>
-      <mass value="${arm_mass}"/>
-      <inertia
-        ixx="0.1"
-        ixy="0.0"
-        ixz="0.0"
-        iyy="0.1"
-        iyz="0.0"
-        izz="0.1"/>
-    </inertial>
-    <buoyancy><compensation>1.0</compensation></buoyancy>
-  </link>
-  <joint name="arm_base_to_arm_hand" type="fixed">
-    <parent link="arm_base"/>
-    <child link="arm_hand"/>
-    <origin rpy="${alpha} 0 0" xyz="0 0 ${arm_base_height/2}"/>
-  </joint>
-  <link name="arm_hook0">
-    <visual>
-      <origin rpy="0 0 0" xyz="0 0 ${-arm_hook_length/2}"/>
-      <geometry>
-        <cylinder radius="${arm_hook_width}" length="${arm_hook_length}"/>
-      </geometry>
-    </visual>
-    <collision>
-      <origin rpy="0 0 0" xyz="0 0 ${-arm_hook_length/2}"/>
-      <geometry>
-        <cylinder radius="${arm_hook_width}" length="${arm_hook_length}"/>
-      </geometry>
-    </collision>
-    <inertial>
-      <origin rpy="0 0 0" xyz="0 0 ${arm_hook_length/2}"/>
-      <mass value="${hook_mass}"/>
-      <inertia
-        ixx="0.1"
-        ixy="0.0"
-        ixz="0.0"
-        iyy="0.1"
-        iyz="0.0"
-        izz="0.1"/>
-    </inertial>
-  </link>
-  <joint name="OpenHook" type="revolute">
-    <parent link="arm_hand"/>
-    <child link="arm_hook0"/>
-    <axis xyz="1 0 0"/>
-    <origin rpy="${PI/2-alpha} 0 0" xyz="0 0 ${arm_hand_length}"/>
-    <dynamics damping="0.8"/>
-    <limit lower="0" upper="${PI/2}" velocity="1" effort="500"/>
-  </joint>
-  <link name="arm_hook1">
-    <visual>
-      <origin rpy="0 0 0" xyz="0 0 ${arm_hook_length/4}"/>
-      <geometry>
-        <cylinder radius="${arm_hook_width}" length="${arm_hook_length/2}"/>
-      </geometry>
-    </visual>
-    <collision>
-      <origin rpy="0 0 0" xyz="0 0 ${arm_hook_length/4}"/>
-      <geometry>
-        <cylinder radius="${arm_hook_width}" length="${arm_hook_length/2}"/>
-      </geometry>
-    </collision>
-    <inertial>
-      <origin rpy="0 0 0" xyz="0 0 ${arm_hook_length/4}"/>
-      <mass value="${hook_mass}"/>
-      <inertia
-        ixx="0.1"
-        ixy="0.0"
-        ixz="0.0"
-        iyy="0.1"
-        iyz="0.0"
-        izz="0.1"/>
-    </inertial>
-  </link>
-  <joint name="hook0_to_hook1" type="fixed">
-    <parent link="arm_hook0"/>
-    <child link="arm_hook1"/>
-    <origin rpy="${11*PI/12} 0 0" xyz="0 0 ${-arm_hook_length}"/>
-  </joint>
+  <xacro:macro name="hook" params="name position">
+    <link name="${name}_base">
+      <visual>
+        <origin rpy="0 0 0" xyz="0 0 0"/>
+        <geometry>
+          <box size="${arm_base_width} ${arm_base_width} ${arm_base_height}"/>
+        </geometry>
+      </visual>
+      <xacro:box_inertial mass="${arm_mass}" length="${arm_base_width}" width="${arm_base_width}" heigth="${arm_base_height}"/>
+      <buoyancy><compensation>1.0</compensation></buoyancy>
+    </link>
+    <joint name="base_link_to_${name}_base" type="fixed">
+      <parent link="base_link"/>
+      <child link="${name}_base"/>
+      <origin rpy="0 0 0" xyz="${position} 0 0.9"/>
+    </joint>
+    <link name="${name}_hand">
+      <visual>
+        <origin rpy="0 0 0" xyz="0 0 ${arm_hand_length/2}"/>
+        <geometry>
+          <cylinder radius="${arm_hand_width}" length="${arm_hand_length}"/>
+        </geometry>
+      </visual>
+      <collision>
+        <origin rpy="0 0 0" xyz="0 0 ${arm_hand_length/2}"/>
+        <geometry>
+          <cylinder radius="${arm_hand_width}" length="${arm_hand_length}"/>
+        </geometry>
+      </collision>
+      <inertial>
+        <origin rpy="0 0 0" xyz="0 0 ${arm_hand_length/2}"/>
+        <mass value="${arm_mass}"/>
+        <inertia
+          ixx="0.1"
+          ixy="0.0"
+          ixz="0.0"
+          iyy="0.1"
+          iyz="0.0"
+          izz="0.1"/>
+      </inertial>
+      <buoyancy><compensation>1.0</compensation></buoyancy>
+    </link>
+    <joint name="${name}_base_to_${name}_hand" type="fixed">
+      <parent link="${name}_base"/>
+      <child link="${name}_hand"/>
+      <origin rpy="${alpha} 0 0" xyz="0 0 ${arm_base_height/2}"/>
+    </joint>
+    <link name="${name}_hook0">
+      <visual>
+        <origin rpy="0 0 0" xyz="0 0 ${-arm_hook_length/2}"/>
+        <geometry>
+          <cylinder radius="${arm_hook_width}" length="${arm_hook_length}"/>
+        </geometry>
+      </visual>
+      <collision>
+        <origin rpy="0 0 0" xyz="0 0 ${-arm_hook_length/2}"/>
+        <geometry>
+          <cylinder radius="${arm_hook_width}" length="${arm_hook_length}"/>
+        </geometry>
+      </collision>
+      <inertial>
+        <origin rpy="0 0 0" xyz="0 0 ${arm_hook_length/2}"/>
+        <mass value="${hook_mass}"/>
+        <inertia
+          ixx="0.1"
+          ixy="0.0"
+          ixz="0.0"
+          iyy="0.1"
+          iyz="0.0"
+          izz="0.1"/>
+      </inertial>
+    </link>
+    <joint name="OpenHook_${name}" type="revolute">
+      <parent link="${name}_hand"/>
+      <child link="${name}_hook0"/>
+      <axis xyz="1 0 0"/>
+      <origin rpy="${PI/2-alpha} 0 0" xyz="0 0 ${arm_hand_length}"/>
+      <dynamics damping="0.8"/>
+      <limit lower="0" upper="${PI/2}" velocity="1" effort="500"/>
+    </joint>
+    <link name="${name}_hook1">
+      <visual>
+        <origin rpy="0 0 0" xyz="0 0 ${arm_hook_length/4}"/>
+        <geometry>
+          <cylinder radius="${arm_hook_width}" length="${arm_hook_length/2}"/>
+        </geometry>
+      </visual>
+      <collision>
+        <origin rpy="0 0 0" xyz="0 0 ${arm_hook_length/4}"/>
+        <geometry>
+          <cylinder radius="${arm_hook_width}" length="${arm_hook_length/2}"/>
+        </geometry>
+      </collision>
+      <inertial>
+        <origin rpy="0 0 0" xyz="0 0 ${arm_hook_length/4}"/>
+        <mass value="${hook_mass}"/>
+        <inertia
+          ixx="0.1"
+          ixy="0.0"
+          ixz="0.0"
+          iyy="0.1"
+          iyz="0.0"
+          izz="0.1"/>
+      </inertial>
+    </link>
+    <joint name="${name}_hook0_to_${name}_hook1" type="fixed">
+      <parent link="${name}_hook0"/>
+      <child link="${name}_hook1"/>
+      <origin rpy="${11*PI/12} 0 0" xyz="0 0 ${-arm_hook_length}"/>
+    </joint>
+  </xacro:macro>
 </robot>

File: urdf/robot.xacro (robot description, xacro)
@@ -71,3 +71,8 @@
   <!-- Include arm -->
   <xacro:include filename="arm.xacro"/>
+  <xacro:hook name="arm0" position="0.4"/>
+  <xacro:hook name="arm1" position="0.2"/>
+  <xacro:hook name="arm2" position="0.0"/>
+  <xacro:hook name="arm3" position="-0.2"/>
+  <xacro:hook name="arm4" position="-0.4"/>
 </robot>
